File: kidoairaku.kicad_pcb (KiCad board)
At the start: 2 copper layers, 142.5 x 76 mm, 191 parts, among them J1 Modulo-Jack, J51 Conn_01x01, J52 Conn_01x01, Q1 IRLML6402, Q51 2N7002, SW1 SW_Push, SW11 SW_Push, SW12 SW_Push, SW13 SW_Push, SW14 SW_Push, SW15 SW_Push, SW16 SW_Push, SW2 SW_Push, SW21 SW_Push, SW22 SW_Push, SW23 SW_Push, SW24 SW_Push, SW25 SW_Push, SW26 SW_Push, SW3 SW_Push, SW31 SW_Push, SW32 SW_Push, SW33 SW_Push, SW34 SW_Push, SW35 SW_Push, SW36 SW_Push, SW4 SW_Push, SW5 SW_Push, SW51 SW_SPDT, SW6 SW_Push, U1 ISP1807breakout-RaspberryPiPi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

Commit message: first production
Parts:
- D1, D11, D12, D13, D14, D15, D16, D2, D21, D22, D23, D24, D25, D26, D3, D31, D32, D33, D34, D35, D36, D4, D5, D51, D55, D6: footprint Diode_SMD:D_SOD-123 -> lib:D_SOD-123
Routing:
- net GND: track 1711.6 -> 1741.3 mm
- net VDD: track 1517.1 -> 1522.0 mm
- net Net-(D184-Pad1): track 5.67 -> 8.52 mm
- net col6: track 246.7 -> 249.3 mm
- net Net-(D204-Pad1): track 96.0 -> 93.5 mm
- net row2: track 130.1 -> 128.4 mm
- net Net-(D208-Pad1): track 88.1 -> 89.5 mm
- net Net-(D113-Pad1): track 6.47 -> 5.22 mm
- net Net-(D211-Pad1): track 15.9 -> 14.8 mm
- net /NeoPixel/NeoPixel: track 222.8 -> 221.7 mm
- net col5: track 214.0 -> 213.0 mm
- net Net-(D111-Pad1): track 162.3 -> 163.2 mm
- net Net-(D157-Pad1): track 130.8 -> 131.5 mm
- net Net-(D202-Pad1): track 17.7 -> 17.1 mm
- net NEOPIXEL: track 26.3 -> 25.6 mm
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